File: audio.kicad_sch (KiCad schematic)
At the start: 9 parts, among them J7 AudioJack3_SwitchTR, U3 LM4950TS

Commit message: save state
Connections:
- net SPI0.MOSI: now reaches DD1.17 (SDIO)
Changed lines of the file:
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@@
+	(wire
+		(pts
+			(xy 177.8 143.51) (xy 167.64 143.51)
+		)
+		(stroke
+			(width 0)
+			(type default)
+		)
+	)
 	(wire
 		(pts
@@
 		(effects
 			(font
+				(size 1.27 1.27)
+			)
+			(justify left bottom)
+		)
+	)
+	(label "SPI0.MOSI"
+		(at 177.8 143.51 0)
+		(effects
+			(font

Commit message: save state
Parts:
- added J10: AudioJack3_SwitchTR, Connector_Audio:Jack_3.5mm_CUI_SJ2-3593D-SMT_Horizontal, symbol Connector_Audio:AudioJack3_SwitchTR
Connections:
- net RFGND: now also J10.S
- new net: J10.R, J10.RN
- new net: J10.T, J10.TN
Changed lines of the file:
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@@
 	(paper "A3")
+	(junction
+		(at 85.09 40.64)
+		(diameter 0)
+		(color 0 0 0 0)
+	)
 	(junction
 		(at 340.36 93.98)
@@
 	)
 	(junction
+		(at 85.09 48.26)
+		(diameter 0)
+		(color 0 0 0 0)
+	)
+	(junction
+		(at 78.74 48.26)
+		(diameter 0)
+		(color 0 0 0 0)
+	)
+	(junction
 		(at 128.27 105.41)
 		(diameter 0)
@@
 	(wire
 		(pts
+			(xy 107.95 40.64) (xy 85.09 40.64)
+		)
+		(stroke
+			(width 0)
+			(type default)
+		)
+	)
+	(wire
+		(pts
 			(xy 68.58 140.97) (xy 109.22 140.97)
 		)
@@
 	(wire
 		(pts
+			(xy 85.09 45.72) (xy 85.09 48.26)
+		)
+		(stroke
+			(width 0)
+			(type default)
+		)
+	)
+	(wire
+		(pts
 			(xy 68.58 143.51) (xy 109.22 143.51)
 		)
@@
 	(wire
 		(pts
+			(xy 119.38 50.8) (xy 78.74 50.8)
+		)
+		(stroke
+			(width 0)
+			(type default)
+		)
+	)
+	(wire
+		(pts
 			(xy 92.71 120.65) (xy 99.06 120.65)
 		)
@@
 	(wire
 		(pts
+			(xy 85.09 43.18) (xy 78.74 43.18)
+		)
+		(stroke
+			(width 0)
+			(type default)
+		)
+	)
+	(wire
+		(pts
 			(xy 180.34 92.71) (xy 135.89 92.71)
 		)
@@
 	(wire
 		(pts
+			(xy 85.09 48.26) (xy 78.74 48.26)
+		)
+		(stroke
+			(width 0)
+			(type default)
+		)
+	)
+	(wire
+		(pts
 			(xy 99.06 168.91) (xy 134.62 168.91)
 		)
@@
 	(wire
 		(pts
+			(xy 78.74 48.26) (xy 77.47 48.26)
+		)
+		(stroke
+			(width 0)
+			(type default)
+		)
+	)
+	(wire
+		(pts
 			(xy 137.16 161.29) (xy 137.16 172.72)
 		)
@@
 	(wire
 		(pts
+			(xy 78.74 45.72) (xy 85.09 45.72)
+		)
+		(stroke
+			(width 0)
+			(type default)
+		)
+	)
+	(wire
+		(pts
 			(xy 177.8 143.51) (xy 167.64 143.51)
 		)
@@
 	(wire
 		(pts
+			(xy 85.09 40.64) (xy 85.09 43.18)
+		)
+		(stroke
+			(width 0)
+			(type default)
+		)
+	)
+	(wire
+		(pts
 			(xy 106.68 181.61) (xy 147.32 181.61)
 		)
@@
 	(wire
 		(pts
+			(xy 113.03 48.26) (xy 85.09 48.26)
+		)
+		(stroke
+			(width 0)
+			(type default)
+		)
+	)
+	(wire
+		(pts
 			(xy 147.32 161.29) (xy 147.32 181.61)
 		)
@@
 	(wire
 		(pts
+			(xy 78.74 40.64) (xy 85.09 40.64)
+		)
+		(stroke
+			(width 0)
+			(type default)
+		)
+	)
+	(wire
+		(pts
 			(xy 312.42 87.63) (xy 312.42 101.6)
 		)
@@
 			(width 0)
 			(type default)
+		)
+	)
+	(label "RFGND"
+		(at 119.38 50.8 0)
+		(effects
+			(font
+				(size 1.27 1.27)
+			)
+			(justify left bottom)
 		)
 	)
@@
 				)
 			)
+		)
+	)
+	(symbol
+		(lib_id "Connector_Audio:AudioJack3_SwitchTR")
+		(at 73.66 48.26 0)
+		(mirror x)
+		(unit 1)
+		(body_style 1)
+		(exclude_from_sim no)
+		(in_bom yes)
+		(on_board yes)
+		(in_pos_files yes)
+		(dnp no)
+		(fields_autoplaced yes)
+		(property "Reference" "J10"
+			(at 66.04 43.8149 0)
+			(show_name no)
+			(do_not_autoplace no)
+			(effects
+				(font
+					(size 1.27 1.27)
+				)
+				(justify right)
+			)
+		)
+		(property "Value" "AudioJack3_SwitchTR"
+			(at 66.04 46.3549 0)
+			(show_name no)
+			(do_not_autoplace no)
+			(effects
+				(font
+					(size 1.27 1.27)
+				)
+				(justify right)
+			)
+		)
+		(property "Footprint" "Connector_Audio:Jack_3.5mm_CUI_SJ2-3593D-SMT_Horizontal"
+			(at 73.66 48.26 0)
+			(hide yes)
+			(show_name no)
+			(do_not_autoplace no)
+			(effects
+				(font
+					(size 1.27 1.27)
+				)
+			)
+		)
+		(property "Datasheet" ""
+			(at 73.66 48.26 0)
+			(hide yes)
+			(show_name no)
+			(do_not_autoplace no)
+			(effects
+				(font
+					(size 1.27 1.27)
+				)
+			)
+		)
+		(property "Description" "Audio Jack, 3 Poles (Stereo / TRS), Switched TR Poles (Normalling)"
+			(at 73.66 48.26 0)
+			(hide yes)
+			(show_name no)
+			(do_not_autoplace no)
+			(effects
+				(font
+					(size 1.27 1.27)
+				)
+			)
+		)
+		(pin "R"
+		)
+		(pin "S"
+		)
+		(pin "T"
+		)
+		(pin "TN"
+		)
+		(pin "RN"
+		)
+		(instances
+			(project "testprj"
+				(path "/ddd61d5c-92f4-4e47-b514-f1213dbaa549"
+					(reference "J10")
+					(unit 1)
+				)
+			)
