File: control.kicad_sch (KiCad schematic)
At the start: 4 parts, among them U4 74HC595, U6 74HC595, U7 74HC595, U8 74HC595

Commit message: save state
Parts:
- added C30, C31, C32, C33: 8200 pF, Capacitor_SMD:C_0805_2012Metric_Pad1.18x1.45mm_HandSolder, symbol Device:C
- added J8, J9: AudioJack3_SwitchTR, Connector_Audio:Jack_3.5mm_CUI_SJ2-3593D-SMT_Horizontal, symbol Connector_Audio:AudioJack3_SwitchTR
- added R10, R11, R12, R13: 100 R, Resistor_SMD:R_0805_2012Metric_Pad1.20x1.40mm_HandSolder, symbol Device:R
- added U10, U9: USBLC6-2SC6, Package_TO_SOT_SMD:SOT-23-6, symbol Power_Protection:USBLC6-2SC6
Connections:
- net RFGND: now also C30.2, C31.1, C32.1, C33.2, J8.S, J9.S, U10.2 (GND), U9.2 (GND)
- new net: J8.R, J8.RN, R11.1
- new net: C31.2, R11.2, U9.3 (I/O2)
- new net: C33.1, R13.2, U10.1 (I/O1)
- new net: C32.2, R12.2, U10.3 (I/O2)
- new net: C30.1, R10.2, U9.1 (I/O1)
- new net: J8.T, J8.TN, R10.1
- new net: J9.R, J9.RN, R12.1
- new net: J9.T, J9.TN, R13.1
