File: testprj.kicad_pcb (KiCad board)
At the start: 4 copper layers, 17 parts, among them J4 Conn_01x40_MountingPin, U2 ST1S10PHR, U5 W25Q128JVE, Y2 Crystal_GND24

Commit message: updates
Parts:
- added C10: C, Capacitor_SMD:C_0805_2012Metric_Pad1.18x1.45mm_HandSolder, F.Cu at (99.2, 128.7)
- added C11: C, Capacitor_SMD:C_0805_2012Metric_Pad1.18x1.45mm_HandSolder, F.Cu at (99.2, 131.7)
- added C14: C, Capacitor_SMD:C_0805_2012Metric_Pad1.18x1.45mm_HandSolder, F.Cu at (99.2, 134.7)
- added C15: C, Capacitor_SMD:C_0805_2012Metric_Pad1.18x1.45mm_HandSolder, F.Cu at (99.2, 137.7)
- added C3: C_Polarized, Capacitor_SMD:CP_Elec_6.3x5.4, F.Cu at (96.7, 109.6)
- added C4: C_Polarized, Capacitor_SMD:CP_Elec_6.3x5.4, F.Cu at (96.7, 117.7)
- added DD1: NAU88C22YG, Package_DFN_QFN:TQFN-32-1EP_5x5mm_P0.5mm_EP3.1x3.1mm_ThermalVias, F.Cu at (74.0, 135.5)
- added J7: AudioJack3_SwitchTR, Connector_Audio:Jack_3.5mm_CUI_SJ2-3593D-SMT_Horizontal, F.Cu at (85.2, 115.0)
- added U3: LM4950TS, Package_TO_SOT_SMD:TO-263-9_TabPin5, F.Cu at (89.8, 133.3)
- added U4: 74HC595, Package_SO:TSSOP-16_4.4x5mm_P0.65mm, F.Cu at (74.8, 108.8)
- added U6: 74HC595, Package_SO:TSSOP-16_4.4x5mm_P0.65mm, F.Cu at (74.8, 115.4)
- added U7: 74HC595, Package_SO:TSSOP-16_4.4x5mm_P0.65mm, F.Cu at (74.8, 122.0)
- added U8: 74HC595, Package_SO:TSSOP-16_4.4x5mm_P0.65mm, F.Cu at (74.8, 128.6)

Commit message: save state
Parts:
- added C25: 2.2 uF, Capacitor_SMD:C_0805_2012Metric_Pad1.18x1.45mm_HandSolder, F.Cu at (153.5, 93.5)
- added C26: 2.2 uF, Capacitor_SMD:C_0805_2012Metric_Pad1.18x1.45mm_HandSolder, F.Cu at (153.5, 96.5)
- added C27: 2.2 uF, Capacitor_SMD:C_0805_2012Metric_Pad1.18x1.45mm_HandSolder, F.Cu at (153.0, 100.0)
- C23, C24: value C -> 22 pF
- moved C23 12.5 mm to (139.0, 70.0)
- moved C24 11.0 mm to (137.5, 73.5)
- moved R8 6.33 mm to (127.5, 76.0)
- moved R7 5.41 mm to (126.5, 73.0)
Connections:
- DD4 pad 107: unconnected-(DD4-VCC-TVIN-Pad107) -> /AVDD_1P8
- DD4 pad 112: unconnected-(DD4-USB1-DP-Pad112) -> /USB1.DM
- DD4 pad 113: unconnected-(DD4-USB1-DM-Pad113) -> /USB1.DP
- DD4 pad 114: unconnected-(DD4-USB0-DM-Pad114) -> /USB0.DM
- DD4 pad 115: unconnected-(DD4-USB0-DP-Pad115) -> /USB0.DP
- DD4 pad 116: unconnected-(DD4-VDD-CORE0-Pad116) -> /SYS_0P95
- DD4 pad 117: unconnected-(DD4-VDD-CORE1-Pad117) -> /SYS_0P95
- DD4 pad 124: unconnected-(DD4-PG12-Pad124) -> /CODEC.WS
- DD4 pad 125: unconnected-(DD4-PG13-Pad125) -> /CODEC.BCLK
- DD4 pad 126: unconnected-(DD4-PG14-Pad126) -> /CODEC.DIN
- DD4 pad 127: unconnected-(DD4-PG15-Pad127) -> /CODEC.DOUT
- DD4 pad 20: unconnected-(DD4-VCC-PLL-Pad20) -> /AVDD_1P8
- DD4 pad 26: unconnected-(DD4-VCC-RTC-Pad26) -> /AVDD_1P8
- DD4 pad 28: unconnected-(DD4-LDOA-OUT-Pad28) -> /AVDD_1P8
- DD4 pad 29: unconnected-(DD4-LDO-IN-Pad29) -> /CPU_VCC3P3
- DD4 pad 30: unconnected-(DD4-LDOB-OUT-Pad30) -> /DRAM_1P5
- DD4 pad 34: unconnected-(DD4-VCC-PE-Pad34) -> /CPU_VCC3P3
- DD4 pad 46: unconnected-(DD4-VDD-SYS0-Pad46) -> /SYS_0P95
- DD4 pad 48: unconnected-(DD4-VCC-DRAM0-Pad48) -> /DRAM_1P5
- DD4 pad 49: unconnected-(DD4-VCC-DRAM1-Pad49) -> /DRAM_1P5
- DD4 pad 50: unconnected-(DD4-VDD18-DRAM-Pad50) -> /AVDD_1P8
- DD4 pad 51: unconnected-(DD4-VDD-SYS1-Pad51) -> /SYS_0P95
- DD4 pad 65: unconnected-(DD4-VCC-LVDS-Pad65) -> /AVDD_1P8
- DD4 pad 66: unconnected-(DD4-VCC-PD-Pad66) -> /CPU_VCC3P3
- DD4 pad 77: unconnected-(DD4-VCC-TVOUT-Pad77) -> /CPU_VCC3P3
- DD4 pad 81: unconnected-(DD4-VDD-SYS2-Pad81) -> /SYS_0P95
- DD4 pad 83: unconnected-(DD4-VCC-IO-Pad83) -> /CPU_VCC3P3
- DD4 pad 89: unconnected-(DD4-AVCC-Pad89) -> /AVDD_1P8
- DD4 pad 90: unconnected-(DD4-VRA2-Pad90) -> Net-(DD4-VRA2)
- DD4 pad 92: unconnected-(DD4-VRA1-Pad92) -> Net-(DD4-VRA1)
- DD4 pad 97: unconnected-(DD4-HPVCC-Pad97) -> Net-(DD4-HPVCC)

Commit message: save state
Parts:
- added C28: 2.2 uF, Capacitor_SMD:C_0805_2012Metric_Pad1.18x1.45mm_HandSolder, F.Cu at (130.5, 124.5)
- added C29: 2.2 uF, Capacitor_SMD:C_0805_2012Metric_Pad1.18x1.45mm_HandSolder, F.Cu at (122.4, 133.5)
- added C30: 8200 pF, Capacitor_SMD:C_0805_2012Metric_Pad1.18x1.45mm_HandSolder, F.Cu at (60.5, 52.0)
- added C31: 8200 pF, Capacitor_SMD:C_0805_2012Metric_Pad1.18x1.45mm_HandSolder, F.Cu at (53.7, 52.2)
- added C32: 8200 pF, Capacitor_SMD:C_0805_2012Metric_Pad1.18x1.45mm_HandSolder, F.Cu at (61.5, 59.5)
- added C33: 8200 pF, Capacitor_SMD:C_0805_2012Metric_Pad1.18x1.45mm_HandSolder, F.Cu at (61.5, 56.5)
- added J10: AudioJack3_SwitchTR, Connector_Audio:Jack_3.5mm_CUI_SJ2-3593D-SMT_Horizontal, F.Cu at (83.6, 84.5)
- added J8: AudioJack3_SwitchTR, Connector_Audio:Jack_3.5mm_CUI_SJ2-3593D-SMT_Horizontal, F.Cu at (59.1, 84.5)
- added J9: AudioJack3_SwitchTR, Connector_Audio:Jack_3.5mm_CUI_SJ2-3593D-SMT_Horizontal, F.Cu at (71.5, 84.5)
- added R10: 100 R, Resistor_SMD:R_0805_2012Metric_Pad1.20x1.40mm_HandSolder, F.Cu at (79.0, 51.5)
- added R11: 100 R, Resistor_SMD:R_0805_2012Metric_Pad1.20x1.40mm_HandSolder, F.Cu at (79.0, 54.5)
- added R12: 100 R, Resistor_SMD:R_0805_2012Metric_Pad1.20x1.40mm_HandSolder, F.Cu at (79.0, 57.5)
- added R13: 100 R, Resistor_SMD:R_0805_2012Metric_Pad1.20x1.40mm_HandSolder, F.Cu at (79.0, 60.4)
- added U1: USBLC6-2SC6, Package_TO_SOT_SMD:SOT-23-6, F.Cu at (160.0, 118.5)
- added U10: USBLC6-2SC6, Package_TO_SOT_SMD:SOT-23-6, F.Cu at (67.4, 58.0)
- added U9: USBLC6-2SC6, Package_TO_SOT_SMD:SOT-23-6, F.Cu at (67.4, 53.3)
- moved J7 34.2 mm to (98.5, 83.5)
Connections:
- DD1 pad 17: unconnected-(DD1-SDIO-Pad17) -> /SPI0.MOSI

Commit message: Перевёл на иерархические схемы
Parts:
- moved C31 95.5 mm to (123.7, 117.3), turned to 0 degrees
- moved C33 91.3 mm to (123.7, 123.3), turned to 0 degrees
- moved U10 90.5 mm to (133.4, 119.8)
- moved U9 90.5 mm to (133.4, 115.2)
- moved C30 88.7 mm to (123.7, 114.3), turned to 0 degrees
- moved C32 87.0 mm to (123.7, 120.3), turned to 0 degrees
- moved U1 84.2 mm to (82.4, 85.8)
- moved R10 79.9 mm to (128.5, 114.3)
- moved R11 79.9 mm to (128.5, 117.2)
- moved R12 79.9 mm to (128.5, 120.2)
- moved R13 79.9 mm to (128.5, 123.1)
- moved C25 79.4 mm to (77.4, 70.8)
- moved C26 79.4 mm to (77.4, 73.8)
- moved C27 79.1 mm to (77.4, 76.8)
- moved J4 75.3 mm to (89.7, 60.0)
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Connections:
- net /AVDD_1P8 renamed /cpu/AVDD_1P8
- net /CODEC.MCLK renamed /audio2/CODEC.MCLK
- net /CODEC1_LHP renamed /audio2/CODEC1_LHP
- net /CODEC1_LMICIN renamed /audio2/CODEC1_LMICIN
- net /CODEC1_LSPK renamed /audio2/CODEC1_LSPK
- net /CODEC1_RHP renamed /audio2/CODEC1_RHP
- net /CODEC1_RSPK renamed /audio2/CODEC1_RSPK
- net /CPU_PWM5 renamed /cpu/CPU_PWM5
- net /CPU_VCC3P3 renamed /cpu/CPU_VCC3P3
- net /DRAM_1P5 renamed /cpu/DRAM_1P5
- net /RFDND renamed /cpu/RFDND
- net /SPI.SCLK renamed /audio2/SPI.SCLK
- net /SPI0.CS0 renamed /cpu/SPI0.CS0
- net /SPI0.HOLD renamed /cpu/SPI0.HOLD
- net /SPI0.MISO renamed /cpu/SPI0.MISO
- net /SPI0.SCLK renamed /cpu/SPI0.SCLK
- net /SPI0.WP renamed /cpu/SPI0.WP
- net /SYS_0P95 renamed /cpu/SYS_0P95
- net /USB0.DM renamed /cpu/USB0.DM
- net /USB0.DP renamed /cpu/USB0.DP
- net /USB1.DM renamed /cpu/USB1.DM
- net /USB1.DP renamed /cpu/USB1.DP
- net /XTAL_IN renamed /cpu/XTAL_IN
- net /XTAL_OUT renamed /cpu/XTAL_OUT
- DD1 pad 10: /CODEC.DIN -> /audio2/CODEC.DIN
- DD1 pad 17: /SPI0.MOSI -> /audio2/SPI0.MOSI
- DD1 pad 7: /CODEC.WS -> /audio2/CODEC.WS
- DD1 pad 8: /CODEC.BCLK -> /audio2/CODEC.BCLK
- DD1 pad 9: /CODEC.DOUT -> /audio2/CODEC.DOUT
- DD4 pad 124: /CODEC.WS -> /cpu/CODEC.WS
- DD4 pad 125: /CODEC.BCLK -> /cpu/CODEC.BCLK
- DD4 pad 126: /CODEC.DIN -> /cpu/CODEC.DIN
- DD4 pad 127: /CODEC.DOUT -> /cpu/CODEC.DOUT
- DD4 pad 17: /SPI0.MOSI -> /cpu/SPI0.MOSI
- U5 pad 5: /SPI0.MOSI -> /cpu/SPI0.MOSI

Commit message: Перевёл на иерархические схемы
Parts:
- moved J4 62.8 mm to (152.4, 62.8), turned to 90 degrees
Connections:
- net /audio2/CODEC.BCLK renamed /audio/CODEC.BCLK
- net /audio2/CODEC.DIN renamed /audio/CODEC.DIN
- net /audio2/CODEC.DOUT renamed /audio/CODEC.DOUT
- net /audio2/CODEC.MCLK renamed /audio/CODEC.MCLK
- net /audio2/CODEC.WS renamed /audio/CODEC.WS
- net /audio2/CODEC1_LHP renamed /audio/CODEC1_LHP
- net /audio2/CODEC1_LMICIN renamed /audio/CODEC1_LMICIN
- net /audio2/CODEC1_LSPK renamed /audio/CODEC1_LSPK
- net /audio2/CODEC1_RHP renamed /audio/CODEC1_RHP
- net /audio2/CODEC1_RSPK renamed /audio/CODEC1_RSPK
- net /audio2/SPI.SCLK renamed /audio/SPI.SCLK
- net /audio2/SPI0.MOSI renamed /audio/SPI0.MOSI
- DD4 pad 52: unconnected-(DD4-PD22-Pad52) -> LCD.PWM
- DD4 pad 53: unconnected-(DD4-PD21-Pad53) -> LCD.VSYNC
- DD4 pad 54: unconnected-(DD4-PD20-Pad54) -> LCD.HSYNC
- DD4 pad 55: unconnected-(DD4-PD0-Pad55) -> LCD.B7
- DD4 pad 57: unconnected-(DD4-PD2-Pad57) -> LCD.B4
- DD4 pad 58: unconnected-(DD4-PD3-Pad58) -> LCD.B5
- DD4 pad 59: unconnected-(DD4-PD4-Pad59) -> LCD.B6
- DD4 pad 60: unconnected-(DD4-PD5-Pad60) -> LCD.B7
- DD4 pad 61: unconnected-(DD4-PD6-Pad61) -> LCD.G2
- DD4 pad 62: unconnected-(DD4-PD7-Pad62) -> LCD.G3
- DD4 pad 63: unconnected-(DD4-PD8-Pad63) -> LCD.G4
- DD4 pad 64: unconnected-(DD4-PD9-Pad64) -> LCD.G5
- DD4 pad 67: unconnected-(DD4-PD10-Pad67) -> LCD.G6
- DD4 pad 68: unconnected-(DD4-PD11-Pad68) -> LCD.G7
- DD4 pad 69: unconnected-(DD4-PD13-Pad69) -> LCD.R3
- DD4 pad 71: unconnected-(DD4-PD14-Pad71) -> LCD.R4
- DD4 pad 72: unconnected-(DD4-PD15-Pad72) -> LCD.R5
- DD4 pad 73: unconnected-(DD4-PD16-Pad73) -> LCD.R6
- DD4 pad 74: unconnected-(DD4-PD17-Pad74) -> LCD.R7
- DD4 pad 75: unconnected-(DD4-PD18-Pad75) -> LCD.CLK
- DD4 pad 76: unconnected-(DD4-PD19-Pad76) -> LCD.DE
- J4 pad 10: unconnected-(J4-Pin_10-Pad10) -> LCD.R5
- J4 pad 11: unconnected-(J4-Pin_11-Pad11) -> LCD.R6
- J4 pad 12: unconnected-(J4-Pin_12-Pad12) -> LCD.R7
- J4 pad 13: unconnected-(J4-Pin_13-Pad13) -> LCD.G6
- J4 pad 14: unconnected-(J4-Pin_14-Pad14) -> LCD.G7
- J4 pad 15: unconnected-(J4-Pin_15-Pad15) -> LCD.G2
- J4 pad 16: unconnected-(J4-Pin_16-Pad16) -> LCD.G3
- J4 pad 17: unconnected-(J4-Pin_17-Pad17) -> LCD.G4
- J4 pad 18: unconnected-(J4-Pin_18-Pad18) -> LCD.G5
- J4 pad 19: unconnected-(J4-Pin_19-Pad19) -> LCD.G6
- J4 pad 20: unconnected-(J4-Pin_20-Pad20) -> LCD.G7
- J4 pad 21: unconnected-(J4-Pin_21-Pad21) -> LCD.B5
- J4 pad 22: unconnected-(J4-Pin_22-Pad22) -> LCD.B6
- J4 pad 23: unconnected-(J4-Pin_23-Pad23) -> LCD.B7
- J4 pad 24: unconnected-(J4-Pin_24-Pad24) -> LCD.B3
- J4 pad 25: unconnected-(J4-Pin_25-Pad25) -> LCD.B4
- J4 pad 26: unconnected-(J4-Pin_26-Pad26) -> LCD.B5
- J4 pad 27: unconnected-(J4-Pin_27-Pad27) -> LCD.B6
- J4 pad 28: unconnected-(J4-Pin_28-Pad28) -> LCD.B7
- J4 pad 29: unconnected-(J4-Pin_29-Pad29) -> RFGND
- J4 pad 3: unconnected-(J4-Pin_3-Pad3) -> RFGND
- J4 pad 30: unconnected-(J4-Pin_30-Pad30) -> LCD.CLK
- J4 pad 31: unconnected-(J4-Pin_31-Pad31) -> VCC_3P3
- J4 pad 32: unconnected-(J4-Pin_32-Pad32) -> LCD.HSYNC
- J4 pad 33: unconnected-(J4-Pin_33-Pad33) -> LCD.VSYNC
- J4 pad 34: unconnected-(J4-Pin_34-Pad34) -> LCD.DE
- J4 pad 35: unconnected-(J4-Pin_35-Pad35) -> VCC_3P3
- J4 pad 36: unconnected-(J4-Pin_36-Pad36) -> RFGND
- J4 pad 37: unconnected-(J4-Pin_37-Pad37) -> /video/TP.X1_M
- J4 pad 38: unconnected-(J4-Pin_38-Pad38) -> /video/TP.Y1_M
- J4 pad 39: unconnected-(J4-Pin_39-Pad39) -> /video/TP.X2_P
- J4 pad 4: unconnected-(J4-Pin_4-Pad4) -> VCC_3P3
- J4 pad 40: unconnected-(J4-Pin_40-Pad40) -> /video/TP.Y2_P
- J4 pad 5: unconnected-(J4-Pin_5-Pad5) -> LCD.R5
- J4 pad 6: unconnected-(J4-Pin_6-Pad6) -> LCD.R6
- J4 pad 7: unconnected-(J4-Pin_7-Pad7) -> LCD.R7
- J4 pad 8: unconnected-(J4-Pin_8-Pad8) -> LCD.R3
- J4 pad 9: unconnected-(J4-Pin_9-Pad9) -> LCD.R4

Commit message: Добавил клавиатуру
Parts:
- added C17: 22 uF, Capacitor_SMD:C_1206_3216Metric_Pad1.33x1.80mm_HandSolder, F.Cu at (82.0, 53.7)
- added U11: MCP3208, Package_SO:SOIC-16_3.9x9.9mm_P1.27mm, F.Cu at (107.2, 143.9)

Commit message: кнопки
Parts:
- added SW1: SW_Push, Button_Switch_THT:SW_PUSH_6mm_H9.5mm, F.Cu at (74.5, 143.0)
- added SW2: SW_Push, Button_Switch_THT:SW_PUSH_6mm_H9.5mm, F.Cu at (74.5, 151.6)

Commit message: кнопки
Parts:
- added C34: 8200 pF, Capacitor_SMD:C_0805_2012Metric_Pad1.18x1.45mm_HandSolder, F.Cu at (195.4, 132.2)
- added C35: 8200 pF, Capacitor_SMD:C_0805_2012Metric_Pad1.18x1.45mm_HandSolder, F.Cu at (195.4, 135.2)
- added C36: 8200 pF, Capacitor_SMD:C_0805_2012Metric_Pad1.18x1.45mm_HandSolder, F.Cu at (195.4, 138.2)
- added C37: 8200 pF, Capacitor_SMD:C_0805_2012Metric_Pad1.18x1.45mm_HandSolder, F.Cu at (195.4, 141.2)
- added C38: 8200 pF, Capacitor_SMD:C_0805_2012Metric_Pad1.18x1.45mm_HandSolder, F.Cu at (195.4, 144.2)
- added R14: 6K8 F, Resistor_SMD:R_0805_2012Metric_Pad1.20x1.40mm_HandSolder, F.Cu at (176.4, 132.2)
- added R15: 2K2 F, Resistor_SMD:R_0805_2012Metric_Pad1.20x1.40mm_HandSolder, F.Cu at (176.4, 135.1)
- added R16: 4K7 F, Resistor_SMD:R_0805_2012Metric_Pad1.20x1.40mm_HandSolder, F.Cu at (176.4, 138.1)
- added R17: 13K F, Resistor_SMD:R_0805_2012Metric_Pad1.20x1.40mm_HandSolder, F.Cu at (176.4, 141.0)
- added R18: 6K8 F, Resistor_SMD:R_0805_2012Metric_Pad1.20x1.40mm_HandSolder, F.Cu at (176.4, 144.0)
- added R19: 2K2 F, Resistor_SMD:R_0805_2012Metric_Pad1.20x1.40mm_HandSolder, F.Cu at (181.1, 132.2)
- added R20: 4K7 F, Resistor_SMD:R_0805_2012Metric_Pad1.20x1.40mm_HandSolder, F.Cu at (181.1, 135.1)
- added R21: 13K F, Resistor_SMD:R_0805_2012Metric_Pad1.20x1.40mm_HandSolder, F.Cu at (181.1, 138.1)
- added R22: 6K8 F, Resistor_SMD:R_0805_2012Metric_Pad1.20x1.40mm_HandSolder, F.Cu at (181.1, 141.0)
- added R23: 2K2 F, Resistor_SMD:R_0805_2012Metric_Pad1.20x1.40mm_HandSolder, F.Cu at (181.1, 144.0)
- added R24: 4K7 F, Resistor_SMD:R_0805_2012Metric_Pad1.20x1.40mm_HandSolder, F.Cu at (185.9, 132.2)
- added R25: 13K F, Resistor_SMD:R_0805_2012Metric_Pad1.20x1.40mm_HandSolder, F.Cu at (185.9, 135.1)
- added R26: 6K8 F, Resistor_SMD:R_0805_2012Metric_Pad1.20x1.40mm_HandSolder, F.Cu at (185.9, 138.1)
- added R27: 2K2 F, Resistor_SMD:R_0805_2012Metric_Pad1.20x1.40mm_HandSolder, F.Cu at (185.9, 141.0)
- added R28: 4K7 F, Resistor_SMD:R_0805_2012Metric_Pad1.20x1.40mm_HandSolder, F.Cu at (185.9, 144.0)
- added R29: 13K F, Resistor_SMD:R_0805_2012Metric_Pad1.20x1.40mm_HandSolder, F.Cu at (190.6, 132.2)
- added R30: 6K8 F, Resistor_SMD:R_0805_2012Metric_Pad1.20x1.40mm_HandSolder, F.Cu at (190.6, 135.1)
- added R31: 2K2 F, Resistor_SMD:R_0805_2012Metric_Pad1.20x1.40mm_HandSolder, F.Cu at (190.6, 138.1)
- added R32: 4K7 F, Resistor_SMD:R_0805_2012Metric_Pad1.20x1.40mm_HandSolder, F.Cu at (190.6, 141.0)
- added R33: 13K F, Resistor_SMD:R_0805_2012Metric_Pad1.20x1.40mm_HandSolder, F.Cu at (190.6, 144.0)
- added SW10: SW_Push, Button_Switch_THT:SW_PUSH_6mm_H9.5mm, F.Cu at (197.1, 107.1)
- added SW11: SW_Push, Button_Switch_THT:SW_PUSH_6mm_H9.5mm, F.Cu at (197.1, 115.6)
- added SW12: SW_Push, Button_Switch_THT:SW_PUSH_6mm_H9.5mm, F.Cu at (197.1, 124.2)
- added SW13: SW_Push, Button_Switch_THT:SW_PUSH_6mm_H9.5mm, F.Cu at (207.7, 98.5)
- added SW14: SW_Push, Button_Switch_THT:SW_PUSH_6mm_H9.5mm, F.Cu at (207.7, 107.1)
- added SW15: SW_Push, Button_Switch_THT:SW_PUSH_6mm_H9.5mm, F.Cu at (207.7, 115.6)
- added SW16: SW_Push, Button_Switch_THT:SW_PUSH_6mm_H9.5mm, F.Cu at (207.7, 124.2)
- added SW17: SW_Push, Button_Switch_THT:SW_PUSH_6mm_H9.5mm, F.Cu at (218.2, 98.5)
- added SW18: SW_Push, Button_Switch_THT:SW_PUSH_6mm_H9.5mm, F.Cu at (218.2, 107.1)
- added SW19: SW_Push, Button_Switch_THT:SW_PUSH_6mm_H9.5mm, F.Cu at (218.2, 115.6)
- added SW20: SW_Push, Button_Switch_THT:SW_PUSH_6mm_H9.5mm, F.Cu at (218.2, 124.2)
- added SW3: SW_Push, Button_Switch_THT:SW_PUSH_6mm_H9.5mm, F.Cu at (176.0, 115.6)
- added SW4: SW_Push, Button_Switch_THT:SW_PUSH_6mm_H9.5mm, F.Cu at (176.0, 124.2)
- added SW5: SW_Push, Button_Switch_THT:SW_PUSH_6mm_H9.5mm, F.Cu at (186.6, 98.5)
- added SW6: SW_Push, Button_Switch_THT:SW_PUSH_6mm_H9.5mm, F.Cu at (186.6, 107.1)
- added SW7: SW_Push, Button_Switch_THT:SW_PUSH_6mm_H9.5mm, F.Cu at (186.6, 115.6)
- added SW8: SW_Push, Button_Switch_THT:SW_PUSH_6mm_H9.5mm, F.Cu at (186.6, 124.2)
- added SW9: SW_Push, Button_Switch_THT:SW_PUSH_6mm_H9.5mm, F.Cu at (197.1, 98.5)
- moved SW1 110.8 mm to (176.0, 98.5)
- moved SW2 110.8 mm to (176.0, 107.1)
- moved U11 95.1 mm to (202.0, 136.6)
Connections:
- SW1 pad 2: unconnected-(SW1-Pad2) -> /keyboard/KI0
- SW2 pad 2: unconnected-(SW2-Pad2) -> Net-(R15-Pad1)
- U11 pad 1: unconnected-(U11-CH0-Pad1) -> /keyboard/KI0
- U11 pad 2: unconnected-(U11-CH1-Pad2) -> /keyboard/KI1
- U11 pad 3: unconnected-(U11-CH2-Pad3) -> /keyboard/KI2
- U11 pad 4: unconnected-(U11-CH3-Pad4) -> /keyboard/KI3
- U11 pad 5: unconnected-(U11-CH4-Pad5) -> /keyboard/KI4
