File: testprj.kicad_pcb (KiCad board)
At the start: 4 copper layers, 96 parts, among them J10 AudioJack3_SwitchTR, J4 Conn_01x40_MountingPin, J7 AudioJack3_SwitchTR, J8 AudioJack3_SwitchTR, J9 AudioJack3_SwitchTR, SW1 SW_Push, SW10 SW_Push, SW11 SW_Push, SW12 SW_Push, SW13 SW_Push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

Commit message: save state (add 1g logic)
Parts:
- added U12: SN74LVC1G125DBV, Package_TO_SOT_SMD:SOT-23-5, F.Cu at (106.6, 133.9)
- added U13: 74LVC1G32, Package_TO_SOT_SMD:SOT-23-5, F.Cu at (105.1, 144.9)
