File: testprj.kicad_sch (KiCad schematic)
At the start: 18 parts, among them J4 Conn_01x40_MountingPin, U2 ST1S10PHR, U5 W25Q128JVE, Y2 Crystal_GND24

Commit message: updates
Changed lines of the file:
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@@
+		)
+	)
+	(label "CODEC.WS"
+		(at 190.5 77.47 0)
+		(effects
+			(font
+				(size 1.27 1.27)
+			)
+			(justify left bottom)
 		)
 	)
@@
 		)
 	)
+	(label "CODEC.BCLK"
+		(at 190.5 80.01 0)
+		(effects
+			(font
+				(size 1.27 1.27)
+			)
+			(justify left bottom)
+		)
+	)
 	(label "XTAL_OUT"
 		(at 204.47 132.08 0)
@@
 		)
 	)
+	(label "CODEC.MCLK"
+		(at 190.5 87.63 0)
+		(effects
+			(font
+				(size 1.27 1.27)
+			)
+			(justify left bottom)
+		)
+	)
 	(label "SPI0.SCLK"
 		(at 30.48 44.45 0)
@@
 		)
 	)
+	(label "CODEC.DIN"
+		(at 190.5 85.09 0)
+		(effects
+			(font
+				(size 1.27 1.27)
+			)
+			(justify left bottom)
+		)
+	)
 	(label "SPI0.HOLD"
 		(at 195.58 111.76 0)
@@
 		)
 	)
+	(label "CODEC.DOUT"
+		(at 190.5 82.55 0)
+		(effects
+			(font
+				(size 1.27 1.27)
+			)
+			(justify left bottom)
+		)
+	)

Commit message: save state
Parts:
- added C25, C26, C27, C28, C29: 2.2 uF, Capacitor_SMD:C_0805_2012Metric_Pad1.18x1.45mm_HandSolder, symbol Device:C
- C23, C24: value C -> 22 pF
Connections:
- net CODEC.BCLK: now also DD4.125 (PG13)
- net CODEC.DIN: now also DD4.126 (PG14)
- net CODEC.DOUT: now also DD4.127 (PG15)
- net CODEC.WS: now also DD4.124 (PG12)
- net CPU_VCC3P3: now also DD4.29 (LDO-IN), DD4.34 (VCC-PE), DD4.66 (VCC-PD), DD4.77 (VCC-TVOUT), DD4.83 (VCC-IO)
- net RFDND: now also C25.2, C26.2, C27.2
- net RFGND: now also C28.2, C29.2
- net AVDD_1P8: now reaches DD4.107 (VCC-TVIN)
- net AVDD_1P8: now also DD4.20 (VCC-PLL), DD4.26 (VCC-RTC), DD4.28 (LDOA-OUT), DD4.50 (VDD18-DRAM), DD4.65 (VCC-LVDS), DD4.89 (AVCC), C28.1
- net USB1.DM: now reaches DD4.112 (USB1-DP)
- net USB1.DP: now reaches DD4.113 (USB1-DM)
- net USB0.DM: now reaches DD4.114 (USB0-DM)
- net USB0.DP: now reaches DD4.115 (USB0-DP)
- net SYS_0P95: now reaches DD4.116 (VDD-CORE0)
- net SYS_0P95: now also DD4.117 (VDD-CORE1), DD4.46 (VDD-SYS0), DD4.51 (VDD-SYS1), DD4.81 (VDD-SYS2)
- net DRAM_1P5: now reaches DD4.30 (LDOB-OUT)
- net DRAM_1P5: now also DD4.48 (VCC-DRAM0), DD4.49 (VCC-DRAM1), C29.1
- net at DD4.90 (VRA2): now also C27.1
- net at DD4.92 (VRA1): now also C26.1
- net at DD4.97 (HPVCC): now also C25.1
Other:
- moved on the sheet: C16, C17, C18, C19, C20, C21, C22, L5, R7, R8, U2, U5

Commit message: save state
Parts:
- added U1: USBLC6-2SC6, Package_TO_SOT_SMD:SOT-23-6, symbol Power_Protection:USBLC6-2SC6
Connections:
- net RFGND: now also U1.2 (GND)
Changed lines of the file:
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@@
+	(wire
+		(pts
+			(xy 83.82 160.02) (xy 93.98 160.02)
+		)
+		(stroke
+			(width 0)
+			(type default)
+		)
+	)
 	(wire
 		(pts
@@
 	(label "CODEC.DOUT"
 		(at 245.11 46.99 90)
+		(effects
+			(font
+				(size 1.27 1.27)
+			)
+			(justify left bottom)
+		)
+	)
+	(label "RFGND"
+		(at 93.98 160.02 0)
 		(effects
 			(font
@@
 					(unit 1)
 				)
+			)
+		)
+	)
+	(symbol
+		(lib_id "Power_Protection:USBLC6-2SC6")
+		(at 83.82 152.4 0)
+		(unit 1)
+		(body_style 1)
+		(exclude_from_sim no)
+		(in_bom yes)
+		(on_board yes)
+		(in_pos_files yes)
+		(dnp no)
+		(fields_autoplaced yes)
+		(property "Reference" "U1"
+			(at 85.4711 144.78 0)
+			(show_name no)
+			(do_not_autoplace no)
+			(effects
+				(font
+					(size 1.27 1.27)
+				)
+				(justify left)
+			)
+		)
+		(property "Value" "USBLC6-2SC6"
+			(at 85.4711 147.32 0)
+			(show_name no)
+			(do_not_autoplace no)
+			(effects
+				(font
+					(size 1.27 1.27)
+				)
+				(justify left)
+			)
+		)
+		(property "Footprint" "Package_TO_SOT_SMD:SOT-23-6"
+			(at 85.09 158.75 0)
+			(hide yes)
+			(show_name no)
+			(do_not_autoplace no)
+			(effects
+				(font
+					(size 1.27 1.27)
+					(italic yes)
+				)
+				(justify left)
+			)
+		)
+		(property "Datasheet" "https://www.st.com/resource/en/datasheet/usblc6-2.pdf"
+			(at 85.09 160.655 0)
+			(hide yes)
+			(show_name no)
+			(do_not_autoplace no)
+			(effects
+				(font
+					(size 1.27 1.27)
+				)
+				(justify left)
+			)
+		)
+		(property "Description" "Very low capacitance ESD protection diode, 2 data-line, SOT-23-6"
+			(at 83.82 152.4 0)
+			(hide yes)
+			(show_name no)
+			(do_not_autoplace no)
+			(effects
+				(font
+					(size 1.27 1.27)
+				)
+			)
+		)
+		(pin "1"
+		)
+		(pin "3"
+		)
+		(pin "4"
+		)
+		(pin "5"
+		)
+		(pin "2"
+		)
+		(pin "6"
+		)
+		(instances
+			(project "testprj"
+				(path "/423c1216-1c87-4878-aa19-5de0f026118b"
+					(reference "U1")
+					(unit 1)
+				)

Commit message: Перевёл на иерархические схемы
Parts:
- removed C16, C18, C19, C20, C21, C22: 22 uF, Capacitor_SMD:C_1206_3216Metric_Pad1.33x1.80mm_HandSolder, symbol Device:C
- removed C17: 22 uF, symbol Device:C
- removed C23, C24: 22 pF, Capacitor_SMD:C_0805_2012Metric_Pad1.18x1.45mm_HandSolder, symbol Device:C
- removed C25, C26, C27, C28, C29: 2.2 uF, Capacitor_SMD:C_0805_2012Metric_Pad1.18x1.45mm_HandSolder, symbol Device:C
- removed DD4: T113s3, projectlib:TQFP-128_14x14mm_P0.4mm_EP8x8mm, symbol H616_lib:T113s3
- removed J4: Conn_01x40_MountingPin, Connector_FFC-FPC:Amphenol_F32R-1A7x1-11040_1x40-1MP_P0.5mm_Horizontal, symbol Connector_Generic_MountingPin:Conn_01x40_MountingPin
- removed L5: L, Inductor_SMD:L_TDK_VLS6045EX_VLS6045AF, symbol Device:L
- removed R7, R8: R, Resistor_SMD:R_0805_2012Metric_Pad1.20x1.40mm_HandSolder, symbol Device:R
- removed R9: 240 R F, Resistor_SMD:R_0805_2012Metric_Pad1.20x1.40mm_HandSolder, symbol Device:R
- removed U1: USBLC6-2SC6, Package_TO_SOT_SMD:SOT-23-6, symbol Power_Protection:USBLC6-2SC6
- removed U2: ST1S10PHR, Package_SO:TI_SO-PowerPAD-8, symbol Regulator_Switching:ST1S10PHR
- removed U5: W25Q128JVE, Package_SON:WSON-8-1EP_8x6mm_P1.27mm_EP3.4x4.3mm, symbol Memory_Flash:W25Q128JVE
- removed Y2: Crystal_GND24, Crystal:Crystal_SMD_7050-4Pin_7.0x5.0mm, symbol Device:Crystal_GND24
Other:
- added sheet audio2 (audio2.kicad_sch)
- added sheet control2 (control2.kicad_sch)
- added sheet cpu (cpu.kicad_sch)

Commit message: Перевёл на иерархические схемы
Other:
- sheet audio2 renamed audio
- sheet control2 renamed control
- added sheet video (video.kicad_sch)
Changed lines of the file:
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@@
 			(color 0 0 0 0)
 		)
-		(property "Sheetname" "audio2"
+		(property "Sheetname" "audio"
 			(at 58.42 99.6184 0)
 			(show_name no)
@@
 			(color 0 0 0 0)
 		)
-		(property "Sheetname" "control2"
+		(property "Sheetname" "control"
 			(at 62.23 164.3884 0)
 			(show_name no)
@@
 				)
 			)
+		)
+	)
+	(sheet
+		(at 63.5 233.68)
+		(size 113.03 38.1)
+		(exclude_from_sim no)
+		(in_bom yes)
+		(on_board yes)
+		(dnp no)
+		(fields_autoplaced yes)
+		(stroke
+			(width 0.1524)
+			(type solid)
+		)
+		(fill
+			(color 0 0 0 0)
+		)
+		(property "Sheetname" "video"
+			(at 63.5 232.9684 0)
+			(show_name no)
+			(do_not_autoplace no)
+			(effects
+				(font
+					(size 1.27 1.27)
+				)
+				(justify left bottom)
+			)
+		)
+		(property "Sheetfile" "video.kicad_sch"
+			(at 63.5 272.3646 0)
+			(show_name no)
+			(do_not_autoplace no)
+			(effects
+				(font
+					(size 1.27 1.27)
+				)
+				(justify left top)
+			)
+		)
+		(instances
+			(project "testprj"
+				(path "/423c1216-1c87-4878-aa19-5de0f026118b"
+					(page "2")
+				)
+			)

Commit message: Добавил клавиатуру
Other:
- added sheet keyboard (keyboard.kicad_sch)
Changed lines of the file:
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@@
 	)
 	(sheet
-		(at 62.23 165.1)
+		(at 228.6 45.72)
 		(size 107.95 40.64)
 		(exclude_from_sim no)
@@
 		)
 		(property "Sheetname" "control"
-			(at 62.23 164.3884 0)
+			(at 228.6 45.0084 0)
 			(show_name no)
 			(do_not_autoplace no)
@@
 		)
 		(property "Sheetfile" "control2.kicad_sch"
-			(at 62.23 206.3246 0)
+			(at 228.6 86.9446 0)
 			(show_name no)
 			(do_not_autoplace no)
@@
 	)
 	(sheet
-		(at 63.5 233.68)
+		(at 229.87 114.3)
 		(size 113.03 38.1)
 		(exclude_from_sim no)
@@
 		)
 		(property "Sheetname" "video"
-			(at 63.5 232.9684 0)
+			(at 229.87 113.5884 0)
 			(show_name no)
 			(do_not_autoplace no)
@@
 		)
 		(property "Sheetfile" "video.kicad_sch"
-			(at 63.5 272.3646 0)
+			(at 229.87 152.9846 0)
 			(show_name no)
 			(do_not_autoplace no)
@@
 				)
 			)
+		)
+	)
+	(sheet
+		(at 62.23 163.83)
+		(size 101.6 38.1)
+		(exclude_from_sim no)
+		(in_bom yes)
+		(on_board yes)
+		(dnp no)
+		(fields_autoplaced yes)
+		(stroke
+			(width 0.1524)
+			(type solid)
+		)
+		(fill
+			(color 0 0 0 0)
+		)
+		(property "Sheetname" "keyboard"
+			(at 62.23 163.1184 0)
+			(show_name no)
+			(do_not_autoplace no)
+			(effects
+				(font
+					(size 1.27 1.27)
+				)
+				(justify left bottom)
+			)
+		)
+		(property "Sheetfile" "keyboard.kicad_sch"
+			(at 62.23 202.5146 0)
+			(show_name no)
+			(do_not_autoplace no)
+			(effects
+				(font
+					(size 1.27 1.27)
+				)
+				(justify left top)
+			)
+		)
+		(instances
+			(project "testprj"
+				(path "/423c1216-1c87-4878-aa19-5de0f026118b"
+					(page "3")
+				)
+			)

Commit message: save state
Other:
- added sheet power (power.kicad_sch)
- sheet cpu ports: added LCD{R[2..7] G[1..7] B[2..7] CLK DE VSYNC HSYNC PWM}; removed none
- sheet video ports: added LCD{R[2..7] G[1..7] B[2..7] CLK DE VSYNC HSYNC PWM}; removed none
Changed lines of the file:
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@@
 	(generator_version "10.0")
 	(paper "A3")
+	(bus
+		(pts
+			(xy 205.74 124.46) (xy 204.47 57.15)
+		)
+		(stroke
+			(width 0)
+			(type default)
+		)
+	)
+	(bus
+		(pts
+			(xy 204.47 57.15) (xy 158.75 57.15)
+		)
+		(stroke
+			(width 0)
+			(type default)
+		)
+	)
+	(bus
+		(pts
+			(xy 229.87 124.46) (xy 205.74 124.46)
+		)
+		(stroke
+			(width 0)
+			(type default)
+		)
+	)
 	(sheet
 		(at 57.15 46.99)
@@
 			)
 		)
+		(pin "LCD{R[2..7] G[1..7] B[2..7] CLK DE VSYNC HSYNC PWM}" bidirectional
+			(at 158.75 57.15 0)
+			(effects
+				(font
+					(size 1.27 1.27)
+				)
+				(justify right)
+			)
+		)
 		(instances
 			(project "testprj"
@@
 			)
 		)
+		(pin "LCD{R[2..7] G[1..7] B[2..7] CLK DE VSYNC HSYNC PWM}" bidirectional
+			(at 229.87 124.46 180)
+			(effects
+				(font
+					(size 1.27 1.27)
+				)
+				(justify left)
+			)
+		)
 		(instances
 			(project "testprj"
@@
 				)
 			)
+		)
+	)
+	(sheet
+		(at 63.5 232.41)
+		(size 101.6 39.37)
+		(exclude_from_sim no)
+		(in_bom yes)
+		(on_board yes)
+		(dnp no)
+		(fields_autoplaced yes)
+		(stroke
+			(width 0.1524)
+			(type solid)
+		)
+		(fill
+			(color 0 0 0 0)
+		)
+		(property "Sheetname" "power"
+			(at 63.5 231.6984 0)
+			(show_name no)
+			(do_not_autoplace no)
+			(effects
+				(font
+					(size 1.27 1.27)
+				)
+				(justify left bottom)
+			)
+		)
+		(property "Sheetfile" "power.kicad_sch"
+			(at 63.5 272.3646 0)
+			(show_name no)
+			(do_not_autoplace no)
+			(effects
+				(font
+					(size 1.27 1.27)
+				)
+				(justify left top)
+			)
+		)
+		(instances
+			(project "testprj"
+				(path "/423c1216-1c87-4878-aa19-5de0f026118b"
+					(page "7")
+				)
+			)
